File: PCB/Gyro/Gyro.kicad_pcb (KiCad board)
At the start: 2 copper layers, 70 x 70 mm, 36 parts, among them J1 JST-PH-SM4-TB, J2 USB-C-Socket-V, J3 Wago, J4 Reset, J5 BTN, J7 TC2030-USB-NL-DS, Q1 CJ2301, Q3 CJ2301, U1 ESP32-S3-MINI-1, U3 TP4054, U4 ME6211C33M5G-N

Commit message: Started
Parts:
- removed J4: Reset, RevK:AA-Pad
- removed J5: BTN, RevK:WAGO-2060-452-998-404
- removed J7: TC2030-USB-NL-DS, RevK:Tag-Connect_TC2030-IDC-NL_2x03_P1.27mm_Vertical
- removed Q3: CJ2301, RevK:SOT-23
- removed R4: 10K, RevK:R_0402
- removed R8: 100K 1%, RevK:R_0402
- removed V4: ~, RevK:VCUT70N
- added C10: 100nF, RevK:C_0402, F.Cu at (103.3, 108.3)
- added C11: 100nF, RevK:C_0402, F.Cu at (100.3, 107.1)
- added C12: 100nF, RevK:C_0402, F.Cu at (97.9, 104.7)
- added C13: 100nF, RevK:C_0402, F.Cu at (96.7, 101.7)
- added C14: 100nF, RevK:C_0402, F.Cu at (96.7, 98.3)
- added C15: 100nF, RevK:C_0402, F.Cu at (97.9, 95.3)
- added C16: 100nF, RevK:C_0402, F.Cu at (100.3, 92.9)
- added C17: 100nF, RevK:C_0402, F.Cu at (103.3, 91.7)
- added C21: 22uF, RevK:C_0603, F.Cu at (98.5, 91.0)
- added C22: 100uF, RevK:C_0805, F.Cu at (118.3, 92.0)
- added C23: 100uF, RevK:C_0805, F.Cu at (118.3, 108.0)
- added C24: 2.2nF, RevK:C_0402, F.Cu at (105.0, 96.5)
- added C25: 100nF, RevK:C_0402, F.Cu at (101.5, 100.0)
- added C27: 10nF, RevK:C_0402, F.Cu at (108.5, 100.0)
- added C3: 100nF, RevK:C_0402, F.Cu at (109.7, 92.9)
- added C4: 100nF, RevK:C_0402, F.Cu at (112.1, 95.3)
- added C6: 100nF, RevK:C_0402, F.Cu at (113.3, 101.7)
- added C7: 100nF, RevK:C_0402, F.Cu at (112.1, 104.7)
- added C8: 100nF, RevK:C_0402, F.Cu at (109.7, 107.1)
- added C9: 100nF, RevK:C_0402, F.Cu at (106.7, 108.3)
- added D10: XL-1010RGBC-WS2812B, RevK:SMD1010, F.Cu at (105.0, 108.5)
- added D11: XL-1010RGBC-WS2812B, RevK:SMD1010, F.Cu at (101.7, 107.9)
- added D12: XL-1010RGBC-WS2812B, RevK:SMD1010, F.Cu at (99.0, 106.0)
- added D13: XL-1010RGBC-WS2812B, RevK:SMD1010, F.Cu at (97.1, 103.3)
- added D14: XL-1010RGBC-WS2812B, RevK:SMD1010, F.Cu at (96.5, 100.0)
- added D15: XL-1010RGBC-WS2812B, RevK:SMD1010, F.Cu at (97.1, 96.7)
- added D16: XL-1010RGBC-WS2812B, RevK:SMD1010, F.Cu at (99.0, 94.0)
- added D17: XL-1010RGBC-WS2812B, RevK:SMD1010, F.Cu at (101.7, 92.1)
- added D18: ~, RevK:DFN1006-2L, F.Cu at (121.0, 101.0)
- added D5: XL-1010RGBC-WS2812B, RevK:SMD1010, F.Cu at (112.9, 96.7)
- added D6: XL-1010RGBC-WS2812B, RevK:SMD1010, F.Cu at (113.5, 100.0)
- added D7: XL-1010RGBC-WS2812B, RevK:SMD1010, F.Cu at (112.9, 103.3)
- added D8: XL-1010RGBC-WS2812B, RevK:SMD1010, F.Cu at (111.0, 106.0)
- added D9: XL-1010RGBC-WS2812B, RevK:SMD1010, F.Cu at (108.3, 107.9)
- added J6: USB-C-Socket-V, RevK:USB-C-Socket-H, F.Cu at (123.3, 95.0)
- added R10: 5K1, RevK:R_0402, F.Cu at (121.0, 99.0)
- added R15: 10K, RevK:R_0402, F.Cu at (115.0, 91.0)
- added R18: 10K, RevK:R_0402, F.Cu at (116.0, 95.5)
- added SW2: SW_SPST, Button_Switch_SMD:SW_Push_1TS009xxxx-xxxx-xxxx_6x6x5mm, F.Cu at (74.0, 100.0)
- added U2: TP4054, RevK:SOT-23-5, F.Cu at (118.3, 104.1)
- added U5: NX6020CAKS, RevK:SOT-363_SC-70-6, F.Cu at (115.0, 93.0)
- added V3: ~, RevK:VCUT70N, F.Cu at (130.0, 100.0)
- C1, C26: value 100uF -> 100nF; footprint RevK:C_0805 -> RevK:C_0402
- C19: value 100nF -> 1uF
- C2: value C_Polarized -> 100nF; footprint RevK:CP_EIA-7343-31_Kemet-D -> RevK:C_0402
- C20: value 22uF -> 100nF; footprint RevK:C_0603 -> RevK:C_0402
- C5: value 1uF -> 100nF
- D1, D3: value ~ -> XL-1010RGBC-WS2812B; footprint RevK:DFN1006-2L -> RevK:SMD1010
- D2: value MBR0530 -> XL-1010RGBC-WS2812B; footprint RevK:D_SOD-123 -> RevK:SMD1010
- D20: value ~ -> MBR0530; footprint RevK:DFN1006-2L -> RevK:D_SOD-123
- J1: value JST-PH-SM4-TB -> Reset; footprint RevK:JST_PH_S2B-PH-SM4-TB_1x02-1MP_P2.00mm_Horizontal -> RevK:AA-Pad; moved to B.Cu
- J2: value USB-C-Socket-V -> TC2030-USB-NL-DS; footprint RevK:USB-C-Socket-H -> RevK:Tag-Connect_TC2030-IDC-NL_2x03_P1.27mm_Vertical; moved to B.Cu
- J3: value Wago -> JST-PH-SM4-TB; footprint RevK:WAGO-2060-453-998-404 -> RevK:JST_PH_S2B-PH-SM4-TB_1x02-1MP_P2.00mm_Horizontal
- R11: value 100K 1% -> 10K
- R2, R3: value 5K1 -> 10K
- R5, R6: value 10K -> 100K 1%
- R9: value 100K 1% -> 5K1
- U3: value TP4054 -> ME6211C33M5G-N
- U4: value ME6211C33M5G-N -> MPU-6050; footprint RevK:SOT-23-5 -> RevK:InvenSense_QFN-24_4x4mm_P0.5mm
- moved J3 37.1 mm to (125.0, 104.5)
- moved J1 30.2 mm to (86.0, 102.5), turned to 180 degrees
- moved D4 29.6 mm to (111.0, 94.0), turned to 180 degrees
- moved R9 26.8 mm to (121.0, 100.0), turned to 0 degrees
- moved V2 23.5 mm to (100.0, 110.5), turned to 180 degrees
- moved C1 23.1 mm to (75.0, 105.0)
- moved D3 22.2 mm to (108.3, 92.1), turned to -157.5 degrees
- moved R11 21.7 mm to (121.0, 91.5), turned to -90 degrees
- moved U3 21.6 mm to (118.2, 95.0)
- moved D1 18.9 mm to (76.6, 105.1)
- moved C5 18.6 mm to (113.3, 98.3), turned to 11.25 degrees
- moved U1 18.5 mm to (85.8, 102.5)
- moved R3 17.8 mm to (120.3, 95.0)
- moved D2 16.8 mm to (105.0, 91.5), turned to -135 degrees
- moved Q1 15.4 mm to (118.3, 100.9), turned to -90 degrees
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Connections:
- C1 pad 1: +3.3V -> VLED
- C19 pad 1: +3.3V -> Net-(U1-EN)
- C2 pad 1: +3.3V -> VLED
- C26 pad 1: VBUS -> Net-(U4-REGOUT)
- C5 pad 1: Net-(U1-EN) -> VLED
- D1 pad 1: GND -> Net-(D1-O)
- D1 pad 2: LED -> VLED
- D2 pad 1: Net-(D2-K) -> Net-(D2-O)
- D2 pad 2: VBUS -> VLED
- D20 pad 1: GND -> VIN
- D20 pad 2: VBAT -> VBUS
- D3 pad 1: GND -> Net-(D3-O)
- D3 pad 2: BTN -> VLED
- D4 pad 1: unconnected-(D4-O-Pad1) -> Net-(D4-O)
- D4 pad 2: +3.3V -> VLED
- D4 pad 4: RGB -> Net-(D3-O)
- J1 pad 2: VBAT -> Net-(J1-Pin_2)
- J3 pad 2: LED -> VBAT
- J3 pad 3: +3.3V -> GND
- Q1 pad 2: Net-(D2-K) -> VIN
- R11 pad 1: VBUS -> Net-(U1-GPIO34)
- R11 pad 2: GND -> VBUS
- R2 pad 1: Net-(J2-CC1) -> GND
- R2 pad 2: GND -> Net-(U2-PROG)
- R3 pad 1: GND -> VBUS
- R3 pad 2: Net-(J2-CC2) -> GND
- R5 pad 1: VBUS -> VBAT
- R5 pad 2: GND -> Net-(R5-Pad2)
- R6 pad 1: +3.3V -> Net-(R5-Pad2)
- R6 pad 2: BTN -> ADC1
- R7 pad 1: Net-(R7-Pad1) -> ADC1
- R7 pad 2: ADC1 -> GND
- R9 pad 1: VBAT -> Net-(J6-CC1)
- R9 pad 2: Net-(R7-Pad1) -> GND
- U1 pad 25: Net-(J4-Pin_2) -> Net-(J1-Pin_2)
- U1 pad 28: unconnected-(U1-GPIO33-Pad28) -> PLED
- U1 pad 29: unconnected-(U1-GPIO34-Pad29) -> Net-(U1-GPIO34)
- U3 pad 1: CHARGING -> VIN
- U3 pad 3: VBAT -> VIN
- U3 pad 4: VBUS -> unconnected-(U3-NC-Pad4)
- U3 pad 5: Net-(U3-PROG) -> +3.3V
- U4 pad 1: Net-(D2-K) -> GND
- U4 pad 2: GND -> unconnected-(U4-NC-Pad2)
- U4 pad 3: Net-(D2-K) -> unconnected-(U4-NC-Pad3)
- U4 pad 5: +3.3V -> unconnected-(U4-NC-Pad5)
Routing:
- net +3.3V: track 101.9 -> 0.00 mm, vias 7 -> 0
- net VBUS: track 64.9 -> 0.00 mm, vias 6 -> 0
- net VLED: track 0.00 -> 56.8 mm, vias 0 -> 16
- net D-: track 47.3 -> 0.00 mm, vias 2 -> 0
- net D+: track 36.3 -> 0.00 mm, vias 2 -> 0
- net VBAT: track 32.8 -> 0.00 mm, vias 4 -> 0
- net GND: track 93.7 -> 64.1 mm, vias 31 -> 20
- net Net-(J2-CC2): track 20.5 -> 0.00 mm, vias 2 -> 0
- net Net-(U1-EN): track 18.7 -> 0.00 mm, vias 2 -> 0
- net BTN: track 18.7 -> 0.00 mm
- net RGB: track 15.7 -> 0.00 mm
- net Net-(D2-K): track 15.5 -> 0.00 mm
- net Net-(J2-CC1): track 15.3 -> 0.00 mm, vias 2 -> 0
- net LED: track 14.6 -> 0.00 mm
- net USB: track 13.5 -> 0.00 mm, vias 2 -> 0
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- added copper zone on B.Cu, net VLED
- added copper zone on F.Cu, net VLED
- removed copper zone on F.Cu, net VBUS
Other:
- board text removed: "${CURRENT_DATE}"
- board text removed: "+"
- board text removed: "-"
- board text removed: "11"
- board text removed: "17 18"
- board text removed: "2"
- board text removed: "3.7V LiPo"
- board text removed: "3V3"
- board text removed: "5"
- board text removed: "5V"
- board text removed: "A"
- board text removed: "BTN"
- board text removed: "CHG USB"
- board text removed: "LED"
- board text removed: "Made in China for Andrews&Arnold Ltd"
- board text removed: "TC2030"
- board text removed: "U"
- board text removed: "ironman.revk.uk"
- board text removed: "®"

Commit message: As ordered
Parts:
- removed V3: ~, RevK:VCUT70N
- Q1: footprint RevK:SOT-23 -> Package_TO_SOT_SMD:SOT-23
- U3: footprint RevK:SOT-23-5 -> Package_TO_SOT_SMD:SOT-23-5
- U5: value NX6020CAKS -> DMC3400SDW
- moved D18 7.77 mm to (128.8, 100.5)
- moved R5 6.13 mm to (94.7, 108.8), turned to 90 degrees
- moved R3 2.90 mm to (120.2, 92.1)
- moved J2 2.69 mm to (114.8, 106.5), turned to -110 degrees
- moved R6 2.57 mm to (94.7, 107.0), turned to 90 degrees
- moved C20 2.15 mm to (95.2, 95.5), turned to 90 degrees
- moved C21 2.06 mm to (97.2, 92.6), turned to 45 degrees
- moved R2 1.75 mm to (115.8, 102.2), turned to -90 degrees
- moved R7 1.25 mm to (94.7, 105.2), turned to 90 degrees
- moved R11 0.61 mm to (121.1, 92.1)
- moved U2 0.36 mm to (118.3, 104.5)
- moved C22 0.25 mm to (118.1, 92.0)
- moved R10 0.25 mm to (121.0, 99.2), turned to 180 degrees
- moved R9 0.25 mm to (121.0, 100.2)
Connections:
- R6 pad 2: ADC1 -> ADC
- R7 pad 1: ADC1 -> ADC
- SW2 pad 1: unconnected-(SW2-A-Pad1) -> Net-(SW2-A)
- SW2 pad 2: unconnected-(SW2-B-Pad2) -> GND
- U1 pad 10: unconnected-(U1-GPIO6-Pad10) -> ADC
- U1 pad 15: LED -> unconnected-(U1-GPIO11-Pad15)
- U1 pad 21: CHARGING -> unconnected-(U1-GPIO17-Pad21)
- U1 pad 22: USB -> unconnected-(U1-GPIO18-Pad22)
- U1 pad 27: unconnected-(U1-GPIO47-Pad27) -> CHARGING
- U1 pad 37: unconnected-(U1-GPIO41-Pad37) -> SDA
- U1 pad 38: unconnected-(U1-GPIO42-Pad38) -> SCL
- U1 pad 6: BTN -> unconnected-(U1-GPIO2-Pad6)
- U1 pad 8: unconnected-(U1-GPIO4-Pad8) -> Net-(SW2-A)
Routing:
- net +3.3V: track 0.00 -> 87.8 mm, vias 0 -> 5
- net GND: track 64.1 -> 148.3 mm, vias 20 -> 41
- net D-: track 0.00 -> 61.0 mm, vias 0 -> 2
- net VBAT: track 0.00 -> 54.9 mm, vias 0 -> 2
- net D+: track 0.00 -> 50.9 mm, vias 0 -> 2
- net Net-(U1-GPIO34): track 0.00 -> 45.3 mm, vias 0 -> 2
- net PLED: track 0.00 -> 44.1 mm, vias 0 -> 2
- net Net-(D1-O): track 1.17 -> 37.6 mm, vias 1 -> 2
- net VLED: track 56.8 -> 91.9 mm, vias 16 -> 18
- net CHARGING: track 0.00 -> 32.2 mm, vias 0 -> 2
- net VBUS: track 0.00 -> 22.6 mm, vias 0 -> 1
- net ADC: track 0.00 -> 19.1 mm, vias 0 -> 2
- net SCL: track 0.00 -> 16.9 mm, vias 0 -> 2
- net SDA: track 0.00 -> 16.0 mm, vias 0 -> 2
- net VIN: track 0.00 -> 11.4 mm
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- added copper zone on F.Cu, net VBUS
Other:
- board text added: "${CURRENT_DATE}"
- board text added: "+"
- board text added: "-"
- board text added: "21"
- board text added: "3.7V LiPo"
- board text added: "4 5 6 33 34 41 42 47"
- board text added: "SW RGB ADC PLED VBUS SDA SCL CHG"
- board text added: "TC2030"
- board text added: "U"
- board text added: "dp.co.uk"

Commit message: ADCL
Connections:
- R7 pad 2: GND -> ADCL
- U1 pad 36: unconnected-(U1-GPIO40-Pad36) -> ADCL
Routing:
- net ADCL: track 0.00 -> 2.16 mm
Other:
- board text added: "40"

Commit message: Tidy
Parts:
- moved C21 21.1 mm to (76.2, 95.2), turned to 90 degrees
- moved C20 17.8 mm to (77.5, 95.8)
- moved R18 0.82 mm to (115.3, 95.0), turned to 180 degrees
- moved R15 0.35 mm to (115.3, 91.0)
Routing:
- net GND: track 148.3 -> 135.1 mm, vias 41 -> 42
- net VBUS: track 22.6 -> 27.6 mm
- net +3.3V: track 87.8 -> 89.5 mm

Commit message: SS
Other:
- board text added: "33"
- board text added: "4 5 6 34 41 42 47"
- board text added: "PWR"
- board text added: "SW LED ADC VBUS SDA SCL CHG"
- board text removed: "4 5 6 33 34 41 42 47"
- board text removed: "SW RGB ADC PLED VBUS SDA SCL CHG"

Commit message: Try the power distribution switches.
Parts:
- removed R15, R18: 10K, RevK:R_0402
- removed U5: DMC3400SDW, RevK:SOT-363_SC-70-6
- added C28: 22uF, RevK:C_0603, F.Cu at (127.3, 101.3)
- added C29: 22uF, RevK:C_0603, F.Cu at (115.0, 105.5)
- added R4: 10K, RevK:R_0402, F.Cu at (76.4, 103.7)
- added U6: ~, RevK:WCSP-4-0.78x0.78, F.Cu at (73.9, 95.3)
- added U7: ~, RevK:WCSP-4-0.78x0.78, F.Cu at (74.9, 95.3)
- U4: footprint RevK:InvenSense_QFN-24_4x4mm_P0.5mm -> Sensor_Motion:InvenSense_QFN-24_4x4mm_P0.5mm
- moved C21 21.6 mm to (97.7, 92.2), turned to 45 degrees
- moved R6 1.66 mm to (94.4, 105.4)
- moved R7 1.66 mm to (94.4, 103.6)
- moved R5 1.66 mm to (94.4, 107.2)
- moved D18 0.18 mm to (128.9, 100.4)
Connections:
- net RGB renamed LED
- C1 pad 1: VLED -> +3.3V
- C10 pad 1: VLED -> +3.3V
- C11 pad 1: VLED -> +3.3V
- C12 pad 1: VLED -> +3.3V
- C13 pad 1: VLED -> +3.3V
- C14 pad 1: VLED -> +3.3V
- C15 pad 1: VLED -> +3.3V
- C16 pad 1: VLED -> +3.3V
- C17 pad 1: VLED -> +3.3V
- C2 pad 1: VLED -> +3.3V
- C3 pad 1: VLED -> +3.3V
- C4 pad 1: VLED -> +3.3V
- C5 pad 1: VLED -> +3.3V
- C6 pad 1: VLED -> +3.3V
- C7 pad 1: VLED -> +3.3V
- C8 pad 1: VLED -> +3.3V
- C9 pad 1: VLED -> +3.3V
- D1 pad 2: VLED -> +3.3V
- D10 pad 2: VLED -> +3.3V
- D11 pad 2: VLED -> +3.3V
- D12 pad 2: VLED -> +3.3V
- D13 pad 2: VLED -> +3.3V
- D14 pad 2: VLED -> +3.3V
- D15 pad 2: VLED -> +3.3V
- D16 pad 2: VLED -> +3.3V
- D17 pad 2: VLED -> +3.3V
- D18 pad 2: VBAT -> Net-(J3-Pin_2)
- D2 pad 2: VLED -> +3.3V
- D3 pad 2: VLED -> +3.3V
- D4 pad 2: VLED -> +3.3V
- D5 pad 2: VLED -> +3.3V
- D6 pad 2: VLED -> +3.3V
- D7 pad 2: VLED -> +3.3V
- D8 pad 2: VLED -> +3.3V
- D9 pad 2: VLED -> +3.3V
- J3 pad 2: VBAT -> Net-(J3-Pin_2)
- SW2 pad 2: GND -> Net-(J3-Pin_2)
- U1 pad 28: PLED -> unconnected-(U1-GPIO33-Pad28)
- U1 pad 7: unconnected-(U1-GPIO3-Pad7) -> PWR
- U1 pad 8: Net-(SW2-A) -> BTN
Routing:
- net VLED: track 91.9 -> 0.00 mm, vias 18 -> 0
- net +3.3V: track 89.5 -> 173.4 mm, vias 5 -> 23
- net Net-(J3-Pin_2): track 0.00 -> 79.4 mm, vias 0 -> 2
- net VBAT: track 54.9 -> 114.3 mm, vias 2 -> 5
- net PLED: track 44.5 -> 0.00 mm, vias 2 -> 0
- net PWR: track 0.00 -> 13.3 mm
- net Net-(SW2-A): track 4.25 -> 16.4 mm, vias 0 -> 2
- net VIN: track 11.5 -> 7.17 mm
- net BTN: track 0.00 -> 2.35 mm
- net Net-(U5A-D): track 1.84 -> 0.00 mm
- net CHARGING: track 32.2 -> 33.9 mm
- net Net-(U1-GPIO34): track 45.3 -> 46.5 mm
- net D+: track 50.9 -> 52.0 mm
- net GND: track 135.1 -> 136.1 mm, vias 42 -> 46
- net ADC: track 19.1 -> 19.9 mm
- added copper zone on B.Cu, net +3.3V
- added copper zone on F.Cu, net +3.3V
- removed copper zone on B.Cu, net VLED
- removed copper zone on F.Cu, net VLED
