File: PCB/Gyro/Gyro.kicad_pcb (KiCad board)
At the start: 2 copper layers, 70 x 70 mm, 72 parts, among them J1 Reset, J2 TC2030-USB-NL-DS, J3 JST-PH-SM4-TB, J6 USB-C-Socket-V, Q1 CJ2301, SW2 SW_SPST, U1 ESP32-S3-MINI-1, U2 TP4054, U3 ME6211C33M5G-N, U4 MPU-6050

Commit message: Tweaks
Parts:
- R2: value 10K -> 5K1
- moved C21 18.0 mm to (115.7, 93.7), turned to -90 degrees
- moved C29 1.15 mm to (115.5, 106.5), turned to -90 degrees
- moved R6 0.79 mm to (94.2, 106.1)
- moved R7 0.79 mm to (94.2, 104.3)
- moved R5 0.79 mm to (94.2, 107.9)
- moved U7 0.56 mm to (75.5, 95.1)
- moved U6 0.28 mm to (74.1, 95.1)
Connections:
- net VIN renamed Net-(D20-K)
Routing:
- net +3.3V: track 173.4 -> 128.5 mm, vias 23 -> 20
- net GND: track 136.1 -> 132.0 mm, vias 46 -> 47
- net ADCL: track 2.15 -> 1.58 mm
Other:
- board text added: "3 4 5 6 34 41 42 47"
- board text added: "PWR SW LED ADC VBUS SDA SCL CHG"
- board text removed: "33"
- board text removed: "4 5 6 34 41 42 47"
- board text removed: "PWR"
- board text removed: "SW LED ADC VBUS SDA SCL CHG"

Commit message: Tweak SS
Routing:
- net +3.3V: track 128.5 -> 126.6 mm
- net GND: vias 47 -> 49

Commit message: Tweak
Parts:
- Q1: footprint Package_TO_SOT_SMD:SOT-23 -> RevK:SOT-23
- U3: footprint Package_TO_SOT_SMD:SOT-23-5 -> RevK:SOT-23-5
Other:
- board text added: "X"
- board text added: "Y"

Commit message: Tidy
Connections:
- U1 pad 6: unconnected-(U1-GPIO2-Pad6) -> PWR
- U1 pad 7: PWR -> unconnected-(U1-GPIO3-Pad7)
Routing:
- net SDA: track 16.0 -> 17.0 mm
- net Net-(J3-Pin_2): track 79.2 -> 78.6 mm
- net GND: track 132.0 -> 132.1 mm, vias 49 -> 51
Other:
- board text added: "2 4 5 6 34 41 42 47"
- board text removed: "3 4 5 6 34 41 42 47"

Commit message: New power control
Parts:
- removed SW2: SW_SPST, Button_Switch_SMD:SW_Push_1TS009xxxx-xxxx-xxxx_6x6x5mm
- removed U6: ~, RevK:WCSP-4-0.78x0.78
- added SW1: SW_Push_DPDT, RevK:SW_Push_DPDT, F.Cu at (75.0, 100.0)
- moved U7 6.24 mm to (71.3, 99.7), turned to 90 degrees
- moved R4 5.22 mm to (71.6, 101.7), turned to -90 degrees
- moved C20 1.70 mm to (76.4, 94.5), turned to 180 degrees
- moved C1 1.57 mm to (75.7, 106.4)
- moved D1 1.39 mm to (77.0, 106.4), turned to 180 degrees
Connections:
- R4 pad 2: BTN -> PWR
- U4 pad 9: unconnected-(U4-AD0-Pad9) -> GND
Routing:
- net Net-(J3-Pin_2): track 78.6 -> 117.8 mm
- net Net-(U7-ON): track 16.8 -> 5.71 mm, vias 2 -> 0
- net BTN: track 2.35 -> 11.9 mm
- net LED: track 2.29 -> 6.53 mm, vias 0 -> 2
- net PWR: track 13.4 -> 9.26 mm, vias 0 -> 2
- net Net-(D1-O): track 37.2 -> 41.0 mm
- net VBAT: track 113.9 -> 110.8 mm
- net D+: track 52.0 -> 51.1 mm
- net CHARGING: track 33.9 -> 34.6 mm
- net +3.3V: track 126.0 -> 126.6 mm
- net GND: track 132.1 -> 131.8 mm, vias 51 -> 59

Commit message: Render
Parts:
- removed R4: 10K, RevK:R_0402
- added D19: D, RevK:D_0402, F.Cu at (71.6, 101.7)

Commit message: FFS
Connections:
- C28 pad 1: Net-(J3-Pin_2) -> VBAT
- C29 pad 1: VBAT -> VSWITCHED
- D18 pad 2: Net-(J3-Pin_2) -> VBAT
- J3 pad 2: Net-(J3-Pin_2) -> VBAT
- Q1 pad 3: VBAT -> VSWITCHED
- R5 pad 1: VBAT -> VSWITCHED
- SW1 pad 3: Net-(J3-Pin_2) -> VBAT
- U7 pad A1: VBAT -> VSWITCHED
- U7 pad A2: Net-(J3-Pin_2) -> VBAT
Routing:
- net Net-(J3-Pin_2): track 117.8 -> 0.00 mm, vias 2 -> 0
- net VSWITCHED: track 0.00 -> 105.6 mm, vias 0 -> 3
- net VBAT: track 110.8 -> 128.3 mm, vias 5 -> 4
