File: PCB/Gyro/Gyro.kicad_sch (KiCad schematic)
At the start: 36 parts, among them J1 JST-PH-SM4-TB, J2 USB-C-Socket-V, J3 Wago, J4 Reset, J5 BTN, J7 TC2030-USB-NL-DS, Q1 CJ2301, Q3 CJ2301, U1 ESP32-S3-MINI-1, U3 TP4054, U4 ME6211C33M5G-N

Commit message: Started
Parts:
- removed C2: C_Polarized, RevK:CP_EIA-7343-31_Kemet-D, symbol Device:C_Polarized
- removed D1, D3: ~, RevK:DFN1006-2L, symbol RevK:ES05D1MC10
- removed J3: Wago, RevK:WAGO-2060-453-998-404, symbol Connector_Generic:Conn_01x03
- removed J5: BTN, RevK:WAGO-2060-452-998-404, symbol Connector_Generic:Conn_01x02
- removed Q3: CJ2301, RevK:SOT-23, symbol Transistor_FET:BSS83P
- removed R6: 10K, RevK:R_0402, symbol Device:R
- added C1, C10, C11, C12, C13, C14, C15, C16, C17, C2, C25, C26, C3, C4, C5, C6, C7, C8, C9: 100nF, RevK:C_0402, symbol Device:C
- added C24: 2.2nF, RevK:C_0402, symbol Device:C
- added C27: 10nF, RevK:C_0402, symbol Device:C
- added D1, D10, D11, D12, D13, D14, D15, D16, D17, D2, D3, D5, D6, D7, D8, D9: XL-1010RGBC-WS2812B, RevK:SMD1010, symbol RevK:WS2812B-1mm
- added R15, R18: 10K, RevK:R_0402, symbol Device:R
- added SW2: SW_SPST, Button_Switch_SMD:SW_Push_1TS009xxxx-xxxx-xxxx_6x6x5mm, symbol Switch:SW_SPST
- added U4: MPU-6050, RevK:InvenSense_QFN-24_4x4mm_P0.5mm, symbol Sensor_Motion:MPU-6050
- added U5: NX6020CAKS, RevK:SOT-363_SC-70-6, symbol RevK:NX6020CAKS
- R11: value 100K 1% -> 10K; MPN C5139597 -> (none)
- renumbered C5 to C19, C19 to C20, C20 to C21, C1 to C22, C26 to C23, D20 to D18, D2 to D20, J4 to J1, J7 to J2, J1 to J3, J2 to J6, R3 to R10, R4 to R2, R5 to R3, R9 to R5, R7 to R6, R8 to R7, R2 to R9, U3 to U2, U4 to U3, V4 to V2, V2 to V3
Connections:
- net +3.3V: now also C25.1, C27.1, U4.13 (VDD), U4.8 (VLOGIC); no longer D4.2 (+)
- net GND: now also C1.2, C10.2, C11.2, C12.2, C13.2, C14.2, C15.2, C16.2, C17.2, C2.2, C24.2, C25.2, C26.2, C27.2, C3.2, C4.2, C5.2, C6.2, C7.2, C8.2, C9.2, D1.3 (-), D10.3 (-), D11.3 (-), D12.3 (-), D13.3 (-), D14.3 (-), D15.3 (-), D16.3 (-), D17.3 (-), D2.3 (-), D3.3 (-), D5.3 (-), D6.3 (-), D7.3 (-), D8.3 (-), D9.3 (-), R15.1, U4.1 (CLKIN), U4.11 (FSYNC), U4.18 (GND), U5.1 (S); no longer R11.2
- net RGB: now also D1.4 (I); no longer D4.4 (I)
- net VBUS: now also R11.2; no longer R11.1
- net VIN: now reaches D20.1 (K), Q1.2 (S), U3.1 (IN), U3.3 (EN)
- net VIN: now also R18.2, U5.4 (S)
- net at D4.1 (O): now also D5.4 (I)
- net PLED: now reaches U1.28 (GPIO33)
- net PLED: now also R15.2, U5.2 (G)
- net at U1.29 (GPIO34): now also R11.1
- new net: R18.1, U5.5 (G), U5.6 (D)
- new net: D1.1 (O), D2.4 (I)
- new net: D2.1 (O), D3.4 (I)
- new net: D8.1 (O), D9.4 (I)
- new net: D7.1 (O), D8.4 (I)
- new net: D16.1 (O), D17.4 (I)
- new net: D15.1 (O), D16.4 (I)
- new net: D10.1 (O), D11.4 (I)
- new net: D10.4 (I), D9.1 (O)
- new net: C26.1, U4.10 (REGOUT)
- new net: D6.1 (O), D7.4 (I)
- new net: D14.1 (O), D15.4 (I)
- new net: D13.1 (O), D14.4 (I)
- new net: D11.1 (O), D12.4 (I)
- new net: D5.1 (O), D6.4 (I)
- new net: D3.1 (O), D4.4 (I)
- new net: D12.1 (O), D13.4 (I)
- new net: C24.1, U4.20 (CPOUT)
- new net SCL: U4.23 (SCL)
- new net SDA: U4.24 (SDA)
- new net VLED: C1.1, C10.1, C11.1, C12.1, C13.1, C14.1, C15.1, C16.1, C17.1, C2.1, C3.1, C4.1, C5.1, C6.1, C7.1, C8.1, C9.1, D1.2 (+), D10.2 (+), D11.2 (+), D12.2 (+), D13.2 (+), D14.2 (+), D15.2 (+), D16.2 (+), D17.2 (+), D2.2 (+), D3.2 (+), D4.2 (+), D5.2 (+), D6.2 (+), D7.2 (+), D8.2 (+), D9.2 (+), U5.3 (D)
- no-connect marks 31 -> 32
Other:
- title: GPS reference -> (none)
- moved on the sheet: C20, C21, D18, J2, J3

Commit message: As ordered
Parts:
- removed V3: ~, RevK:VCUT70N, symbol RevK:VCUT
- J1: now left out of the parts list
- Q1: footprint RevK:SOT-23 -> Package_TO_SOT_SMD:SOT-23; MPN C5224170 -> C8547
- R1, R11, R15, R18, R2, R3: MPN (none) -> C25744
- R10, R9: MPN (none) -> C25905
- U3: footprint RevK:SOT-23-5 -> Package_TO_SOT_SMD:SOT-23-5; Rotation Offset (none) -> 90
- U4: MPN (none) -> C24112; Rotation Offset (none) -> -90
- U5: value NX6020CAKS -> DMC3400SDW; MPN (none) -> C155499
Connections:
- net ADC1 is gone; now on net ADC: R6.2, R7.1
- net CHARGING: now also U1.27 (GPIO47); no longer U1.21 (GPIO17)
- net GND: now also SW2.2 (B)
- net SCL: now also U1.38 (GPIO42)
- net SDA: now also U1.37 (GPIO41)
- net ADC: now reaches U1.10 (GPIO6)
- net at U1.8 (GPIO4): now also SW2.1 (A)
- net BTN: no longer names the net of U1.6 (GPIO2)
- net LED: no longer names the net of U1.15 (GPIO11)
- net USB: no longer names the net of U1.22 (GPIO18)
Other:
- moved on the sheet: SW2

Commit message: ADCL
Connections:
- net GND: no longer R7.2
- net ADCL: now reaches U1.36 (GPIO40)
- net ADCL: now also R7.2
- no-connect marks 32 -> 31
Other:
- moved on the sheet: D18, J3
Changed lines of the file:
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@@
 	)
 	(junction
-		(at 144.78 57.785)
+		(at 125.095 64.77)
 		(diameter 0)
 		(color 0 0 0 0)
@@
 	)
 	(junction
-		(at 144.78 50.165)
+		(at 125.095 57.15)
 		(diameter 0)
 		(color 0 0 0 0)
@@
 	)
 	(no_connect
-		(at 73.025 68.58)
-	)
-	(no_connect
 		(at 42.545 78.74)
 	)
@@
 	(wire
 		(pts
-			(xy 140.335 62.865) (xy 149.225 62.865)
+			(xy 120.65 69.85) (xy 129.54 69.85)
 		)
 		(stroke
@@
 	(wire
 		(pts
-			(xy 147.955 50.165) (xy 147.955 55.245)
+			(xy 128.27 57.15) (xy 128.27 62.23)
 		)
 		(stroke
@@
 	(wire
 		(pts
-			(xy 147.955 55.245) (xy 149.225 55.245)
+			(xy 128.27 62.23) (xy 129.54 62.23)
 		)
 		(stroke
@@
 	(wire
 		(pts
-			(xy 140.335 57.785) (xy 144.78 57.785)
+			(xy 120.65 64.77) (xy 125.095 64.77)
 		)
 		(stroke
@@
 	(wire
 		(pts
-			(xy 144.78 57.785) (xy 149.225 57.785)
+			(xy 125.095 64.77) (xy 129.54 64.77)
 		)
 		(stroke
@@
 	(wire
 		(pts
-			(xy 140.335 60.325) (xy 149.225 60.325)
+			(xy 120.65 67.31) (xy 129.54 67.31)
 		)
 		(stroke
@@
 	(wire
 		(pts
-			(xy 144.78 50.165) (xy 147.955 50.165)
+			(xy 125.095 57.15) (xy 128.27 57.15)
 		)
 		(stroke
@@
 	(wire
 		(pts
-			(xy 140.335 50.165) (xy 144.78 50.165)
+			(xy 120.65 57.15) (xy 125.095 57.15)
 		)
 		(stroke
@@
 		)
 	)
+	(global_label "ADCL"
+		(shape bidirectional)
+		(at 73.025 68.58 0)
+		(effects
+			(font
+				(size 1.27 1.27)
+			)
+			(justify left)
+		)
+		(property "Intersheetrefs" "${INTERSHEET_REFS}"
+			(at 73.025 68.58 0)
+			(effects
+				(font
+					(size 1.27 1.27)
+				)
+				(hide yes)
+			)
+		)
+	)
 	(global_label "SDA"
 		(shape bidirectional)
@@
 	(global_label "VBAT"
 		(shape bidirectional)
-		(at 140.335 57.785 180)
+		(at 120.65 64.77 180)
 		(fields_autoplaced yes)
 		(effects
@@
 		)
 		(property "Intersheetrefs" "${INTERSHEET_REFS}"
-			(at 132.6367 57.785 0)
+			(at 112.9517 64.77 0)
 			(effects
 				(font
@@
 		)
 	)
+	(global_label "ADCL"
+		(shape bidirectional)
+		(at 219.075 91.44 270)
+		(effects
+			(font
+				(size 1.27 1.27)
+			)
+			(justify right)
+		)
+		(property "Intersheetrefs" "${INTERSHEET_REFS}"
+			(at 219.075 91.44 90)
+			(effects
+				(font
+					(size 1.27 1.27)
+				)
+				(hide yes)
+			)
+		)
+	)
 	(global_label "SCL"
 		(shape output)
@@
 	(symbol
 		(lib_id "power:GND")
-		(at 140.335 50.165 270)
+		(at 120.65 57.15 270)
 		(unit 1)
 		(exclude_from_sim no)
@@
 		(dnp no)
 		(property "Reference" "#PWR014"
-			(at 133.985 50.165 0)
+			(at 114.3 57.15 0)
 			(effects
 				(font
@@
 		)
 		(property "Value" "GND"
-			(at 135.255 50.165 90)
+			(at 115.57 57.15 90)
 			(effects
 				(font
@@
 		)
 		(property "Footprint" ""
-			(at 140.335 50.165 0)
+			(at 120.65 57.15 0)
 			(effects
 				(font
@@
 		)
 		(property "Datasheet" ""
-			(at 140.335 50.165 0)
+			(at 120.65 57.15 0)
 			(effects
 				(font
@@
 		)
 		(property "Description" "Power symbol creates a global label with name \"GND\" , ground"
-			(at 140.335 50.165 0)
+			(at 120.65 57.15 0)
 			(effects
 				(font
@@
 	(symbol
 		(lib_id "power:GND")
-		(at 140.335 62.865 270)
+		(at 120.65 69.85 270)
 		(unit 1)
 		(exclude_from_sim no)
@@
 		(dnp no)
 		(property "Reference" "#PWR016"
-			(at 133.985 62.865 0)
+			(at 114.3 69.85 0)
 			(effects
 				(font
@@
 		)
 		(property "Value" "GND"
-			(at 135.255 62.865 90)
+			(at 115.57 69.85 90)
 			(effects
 				(font
@@
 		)
 		(property "Footprint" ""
-			(at 140.335 62.865 0)
+			(at 120.65 69.85 0)
 			(effects
 				(font
@@
 		)
 		(property "Datasheet" ""
-			(at 140.335 62.865 0)
+			(at 120.65 69.85 0)
 			(effects
 				(font
@@
 		)
 		(property "Description" "Power symbol creates a global label with name \"GND\" , ground"
-			(at 140.335 62.865 0)
+			(at 120.65 69.85 0)
 			(effects
 				(font
@@
 	)
 	(symbol
-		(lib_id "power:GND")
-		(at 219.075 91.44 0)
-		(unit 1)
-		(exclude_from_sim no)
-		(in_bom yes)
-		(on_board yes)
-		(dnp no)
-		(property "Reference" "#PWR027"
-			(at 219.075 97.79 0)
-			(effects
-				(font
-					(size 1.27 1.27)
-				)
-				(hide yes)
-			)
-		)
-		(property "Value" "GND"
-			(at 219.075 95.25 0)
-			(effects
-				(font
-					(size 1.27 1.27)
-				)
-			)
-		)
-		(property "Footprint" ""
-			(at 219.075 91.44 0)
-			(effects
-				(font
-					(size 1.27 1.27)
-				)
-				(hide yes)
-			)
-		)
-		(property "Datasheet" ""
-			(at 219.075 91.44 0)
-			(effects
-				(font
-					(size 1.27 1.27)
-				)
-				(hide yes)
-			)
-		)
-		(property "Description" "Power symbol creates a global label with name \"GND\" , ground"
-			(at 219.075 91.44 0)
-			(effects
-				(font
-					(size 1.27 1.27)
-				)
-				(hide yes)
-			)
-		)
-		(pin "1"
-		)
-		(instances
-			(project "Watchy"
-				(path "/03039abc-65dd-445c-a352-9e386e1f31aa"
-					(reference "#PWR046")
-					(unit 1)
-				)
-			)
-			(project "EPDBat"
-				(path "/46c350bb-7de4-4e81-aafd-4af55e37aab0"
-					(reference "#PWR047")
-					(unit 1)
-				)
-			)
-			(project "Logger"
-				(path "/babeabf2-f3b0-4ed5-8d9e-0215947e6cf3"
-					(reference "#PWR027")
-					(unit 1)
-				)
-			)
-		)
-	)
-	(symbol
 		(lib_id "RevK:ES05D1MC10")
-		(at 144.78 53.975 90)
+		(at 125.095 60.96 90)
 		(unit 1)
 		(exclude_from_sim no)
@@
 		(dnp no)
 		(property "Reference" "D18"
-			(at 138.43 53.975 90)
+			(at 118.745 60.96 90)
 			(effects
 				(font
@@
 		)
 		(property "Value" "~"
-			(at 144.78 53.975 0)
+			(at 125.095 60.96 0)
 			(effects
 				(font
@@
 		)
 		(property "Footprint" "RevK:DFN1006-2L"
-			(at 141.605 53.34 0)
+			(at 121.92 60.325 0)
 			(effects
 				(font
@@
 		)
 		(property "Datasheet" ""
-			(at 144.78 53.975 0)
+			(at 125.095 60.96 0)
 			(effects
 				(font
@@
 		)
 		(property "Description" ""
-			(at 144.78 53.975 0)
+			(at 125.095 60.96 0)
 			(effects
 				(font
@@
 		)
 		(property "MPN" "C5137770"
-			(at 147.955 53.975 0)
+			(at 128.27 60.96 0)
 			(effects
 				(font
@@
 	(symbol
 		(lib_id "Connector_Generic:Conn_01x04")
-		(at 154.305 57.785 0)
+		(at 134.62 64.77 0)
 		(unit 1)
 		(exclude_from_sim no)
@@
 		(dnp no)
 		(property "Reference" "J3"
-			(at 154.305 66.675 0)
+			(at 134.62 73.66 0)
 			(effects
 				(font
@@
 		)
 		(property "Value" "JST-PH-SM4-TB"
-			(at 157.48 51.435 0)
+			(at 137.795 58.42 0)
 			(effects
 				(font
@@
 		)
 		(property "Footprint" "RevK:JST_PH_S2B-PH-SM4-TB_1x02-1MP_P2.00mm_Horizontal"
-			(at 154.305 57.785 0)
+			(at 134.62 64.77 0)
 			(effects
 				(font
@@
 		)
 		(property "Datasheet" "~"
-			(at 154.305 57.785 0)
+			(at 134.62 64.77 0)
 			(effects
 				(font
@@
 		)
 		(property "Description" "Generic connector, single row, 01x04, script generated (kicad-library-utils/schlib/autogen/connector/)"
-			(at 154.305 57.785 0)
+			(at 134.62 64.77 0)
 			(effects
 				(font
@@
 		)
 		(property "MPN" "C295747"
-			(at 154.305 57.785 0)
+			(at 134.62 64.77 0)
 			(effects
 				(font
@@
 	(symbol
 		(lib_id "power:GND")
-		(at 140.335 60.325 270)
+		(at 120.65 67.31 270)
 		(unit 1)
 		(exclude_from_sim no)
@@
 		(dnp no)
 		(property "Reference" "#PWR015"
-			(at 133.985 60.325 0)
+			(at 114.3 67.31 0)
 			(effects
 				(font
@@
 		)
 		(property "Value" "GND"
-			(at 135.255 60.325 90)
+			(at 115.57 67.31 90)
 			(effects
 				(font
@@
 		)
 		(property "Footprint" ""
-			(at 140.335 60.325 0)
+			(at 120.65 67.31 0)
 			(effects
 				(font
@@
 		)
 		(property "Datasheet" ""
-			(at 140.335 60.325 0)
+			(at 120.65 67.31 0)
 			(effects
 				(font
@@
 		)
 		(property "Description" "Power symbol creates a global label with name \"GND\" , ground"
-			(at 140.335 60.325 0)
+			(at 120.65 67.31 0)
 			(effects
 				(font

Commit message: SS
Connections:
- net RGB renamed LED
Changed lines of the file:
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@@
 		)
 	)
-	(global_label "RGB"
+	(global_label "LED"
 		(shape input)
 		(at 111.76 86.995 90)
@@
 		)
 		(property "Intersheetrefs" "${INTERSHEET_REFS}"
-			(at 111.76 80.854 90)
+			(at 111.76 81.2169 90)
 			(effects
 				(font
@@
 		)
 	)
-	(global_label "RGB"
+	(global_label "LED"
 		(shape output)
 		(at 42.545 45.72 180)
@@
 		)
 		(property "Intersheetrefs" "${INTERSHEET_REFS}"
-			(at 36.404 45.72 0)
-			(effects
-				(font
+			(at 36.7669 45.72 0)
+			(effects
+				(font

Commit message: Try the power distribution switches.
Parts:
- removed R15, R18: 10K, RevK:R_0402, symbol Device:R
- removed U5: DMC3400SDW, RevK:SOT-363_SC-70-6, symbol RevK:NX6020CAKS
- added C28, C29: 22uF, RevK:C_0603, symbol Device:C
- added R4: 10K, RevK:R_0402, symbol Device:R
- added U6, U7: ~, RevK:WCSP-4-0.78x0.78, symbol RevK:TPS22916
- U4: footprint RevK:InvenSense_QFN-24_4x4mm_P0.5mm -> Sensor_Motion:InvenSense_QFN-24_4x4mm_P0.5mm
Connections:
- net VLED is gone; now on net +3.3V: C1.1, C10.1, C11.1, C12.1, C13.1, C14.1, C15.1, C16.1, C17.1, C2.1, C3.1, C4.1, C5.1, C6.1, C7.1, C8.1, C9.1, D1.2 (+), D10.2 (+), D11.2 (+), D12.2 (+), D13.2 (+), D14.2 (+), D15.2 (+), D16.2 (+), D17.2 (+), D2.2 (+), D3.2 (+), D4.2 (+), D5.2 (+), D6.2 (+), D7.2 (+), D8.2 (+), D9.2 (+)
- net GND: now also C28.2, C29.2, U6.B1 (GND), U7.B1 (GND); no longer SW2.2 (B)
- net VBAT: now also C29.1, U6.A1 (VOUT), U7.A1 (VOUT); no longer D18.2, J3.2 (Pin_2)
- net PWR: now reaches U1.7 (GPIO3)
- net PWR: now also U6.B2 (ON)
- net at SW2.1 (A): now also R4.1, U7.B2 (ON); no longer U1.8 (GPIO4)
- net PLED: no longer names the net of U1.28 (GPIO33)
- new net: C28.1, D18.2, J3.2 (Pin_2), SW2.2 (B), U6.A2 (VIN), U7.A2 (VIN)
- new net BTN: R4.2, U1.8 (GPIO4)
Other:
- moved on the sheet: C23, D18, J3, J6, R10, R5, R6, R7, R9, SW2

Commit message: Tweaks
Parts:
- R2: value 10K -> 5K1; MPN C25744 -> C25905
Connections:
- net VIN: no longer names the net of D20.1 (K), Q1.2 (S), U3.1 (IN), U3.3 (EN)
Other:
- note added: "5k1 is approx 200mA charge"
- note added: "CHRG Normal: on Full: off Reverse: off No battery: Twinkle"
- moved on the sheet: C24, C25, C26, C27, U4

Commit message: Tweak
Parts:
- Q1: footprint Package_TO_SOT_SMD:SOT-23 -> RevK:SOT-23
- U3: footprint Package_TO_SOT_SMD:SOT-23-5 -> RevK:SOT-23-5
Changed lines of the file:
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@@
 			)
 		)
-		(property "Footprint" "Package_TO_SOT_SMD:SOT-23-5"
+		(property "Footprint" "RevK:SOT-23-5"
 			(at 187.325 24.13 0)
 			(effects
@@
 			)
 		)
-		(property "Footprint" "Package_TO_SOT_SMD:SOT-23"
+		(property "Footprint" "RevK:SOT-23"
 			(at 165.735 27.305 0)
 			(effects

Commit message: Tidy
Connections:
- net PWR: now also U1.6 (GPIO2); no longer U1.7 (GPIO3)
Changed lines of the file:
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@@
 	)
 	(no_connect
-		(at 42.545 38.1)
+		(at 42.545 40.64)
 	)
 	(no_connect
@@
 	(global_label "PWR"
 		(shape output)
-		(at 42.545 40.64 180)
+		(at 42.545 38.1 180)
 		(fields_autoplaced yes)
 		(effects
@@
 		)
 		(property "Intersheetrefs" "${INTERSHEET_REFS}"
-			(at 36.2226 40.64 0)
+			(at 36.2226 38.1 0)
 			(effects
 				(font
