File: PCB/Gyro/Gyro.kicad_sch (KiCad schematic)
At the start: 72 parts, among them J1 Reset, J2 TC2030-USB-NL-DS, J3 JST-PH-SM4-TB, J6 USB-C-Socket-V, Q1 CJ2301, SW2 SW_SPST, U1 ESP32-S3-MINI-1, U2 TP4054, U3 ME6211C33M5G-N, U4 MPU-6050

Commit message: New power control
Parts:
- removed SW2: SW_SPST, Button_Switch_SMD:SW_Push_1TS009xxxx-xxxx-xxxx_6x6x5mm, symbol Switch:SW_SPST
- removed U6: ~, RevK:WCSP-4-0.78x0.78, symbol RevK:TPS22916
- added SW1: SW_Push_DPDT, RevK:SW_Push_DPDT, symbol RevK:SW_Push_DPDT
Connections:
- net BTN: now also SW1.4 (C); no longer R4.2
- net GND: now also U4.9 (AD0), SW1.1 (A), SW1.5 (B)
- net PWR: now also R4.2
- net at C28.1, D18.2, J3.2 (Pin_2)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: now also SW1.3 (C)
- net at R4.1, U7.B2 (ON): now also SW1.2 (B)
Other:
- moved on the sheet: R4, R5, R6, R7, U7

Commit message: Render
Parts:
- removed R4: 10K, RevK:R_0402, symbol Device:R
- added D19: D, RevK:D_0402, symbol Device:D
Connections:
- net PWR: now also D19.2 (A)
- net at SW1.2 (B), U7.B2 (ON): now also D19.1 (K)
Changed lines of the file:
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@@
+	)
+	(symbol
+		(lib_id "Device:D")
+		(at 234.315 136.525 0)
+		(unit 1)
+		(exclude_from_sim no)
+		(in_bom yes)
+		(on_board yes)
+		(dnp no)
+		(property "Reference" "D19"
+			(at 234.188 139.954 0)
+			(effects
+				(font
+					(size 1.27 1.27)
+				)
+			)
+		)
+		(property "Value" "D"
+			(at 234.315 133.5348 0)
+			(effects
+				(font
+					(size 1.27 1.27)
+				)
+			)
+		)
+		(property "Footprint" "RevK:D_0402"
+			(at 234.315 136.525 0)
+			(effects
+				(font
+					(size 1.27 1.27)
+				)
+				(hide yes)
+			)
+		)
+		(property "Datasheet" "~"
+			(at 234.315 136.525 0)
+			(effects
+				(font
+					(size 1.27 1.27)
+				)
+				(hide yes)
+			)
+		)
+		(property "Description" "Diode"
+			(at 234.315 136.525 0)
+			(effects
+				(font
+					(size 1.27 1.27)
+				)
+				(hide yes)
+			)
+		)
+		(property "Sim.Device" "D"
+			(at 234.315 136.525 0)
+			(effects
+				(font
+					(size 1.27 1.27)
+				)
+				(hide yes)
+			)
+		)
+		(property "Sim.Pins" "1=K 2=A"
+			(at 234.315 136.525 0)
+			(effects
+				(font
+					(size 1.27 1.27)
+				)
+				(hide yes)
+			)
+		)
+		(property "MPN" "C28642302"
+			(at 234.315 136.525 0)
+			(effects
+				(font
+					(size 1.27 1.27)
+				)
+				(hide yes)
+			)
+		)
+		(pin "1"
+		)
+		(pin "2"
+		)
+		(instances
+			(project "Gyro"
+				(path "/babeabf2-f3b0-4ed5-8d9e-0215947e6cf3"
+					(reference "D19")
+					(unit 1)
+				)
+			)
+		)
 	)
 	(symbol
@@
 					(unit 1)
 				)
-			)
-		)
-	)
-	(symbol
-		(lib_id "Device:R")
-		(at 234.315 136.525 90)
-		(unit 1)
-		(exclude_from_sim no)
-		(in_bom yes)
-		(on_board yes)
-		(dnp no)
-		(property "Reference" "R4"
-			(at 234.315 134.62 90)
-			(effects
-				(font
-					(size 1.27 1.27)
-				)
-			)
-		)
-		(property "Value" "10K"
-			(at 234.315 136.525 90)
-			(effects
-				(font
-					(size 1.27 1.27)
-				)
-			)
-		)
-		(property "Footprint" "RevK:R_0402"
-			(at 234.315 138.303 90)
-			(effects
-				(font
-					(size 1.27 1.27)
-				)
-				(hide yes)
-			)
-		)
-		(property "Datasheet" "~"
-			(at 234.315 136.525 0)
-			(effects
-				(font
-					(size 1.27 1.27)
-				)
-				(hide yes)
-			)
-		)
-		(property "Description" "Resistor"
-			(at 234.315 136.525 0)
-			(effects
-				(font
-					(size 1.27 1.27)
-				)
-				(hide yes)
-			)
-		)
-		(property "MPN" "C25744"
-			(at 234.315 136.525 90)
-			(effects
-				(font
-					(size 1.27 1.27)
-				)
-				(hide yes)
-			)
-		)
-		(pin "1"
-		)
-		(pin "2"
-		)
-		(instances
-			(project "Gyro"
-				(path "/babeabf2-f3b0-4ed5-8d9e-0215947e6cf3"
-					(reference "R4")
-					(unit 1)
-				)

Commit message: FFS
Connections:
- net VBAT: now also C28.1, D18.2, J3.2 (Pin_2), SW1.3 (C), U7.A2 (VIN); no longer C29.1, Q1.3 (D), R5.1, U7.A1 (VOUT)
- new net VSWITCHED: C29.1, Q1.3 (D), R5.1, U7.A1 (VOUT)
Other:
- moved on the sheet: R5, R6, R7
Changed lines of the file:
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@@
 	)
 	(junction
-		(at 86.36 130.175)
+		(at 85.725 142.24)
 		(diameter 0)
 		(color 0 0 0 0)
@@
 	(wire
 		(pts
+			(xy 213.36 102.235) (xy 213.36 105.41)
+		)
+		(stroke
+			(width 0)
+			(type default)
+		)
+	)
+	(wire
+		(pts
 			(xy 123.19 119.38) (xy 123.19 124.46)
 		)
@@
 	(wire
 		(pts
-			(xy 90.17 130.175) (xy 86.36 130.175)
+			(xy 89.535 142.24) (xy 85.725 142.24)
 		)
 		(stroke
@@
 		)
 	)
+	(global_label "VBAT"
+		(shape input)
+		(at 213.36 102.235 90)
+		(fields_autoplaced yes)
+		(effects
+			(font
+				(size 1.27 1.27)
+			)
+			(justify left)
+		)
+		(property "Intersheetrefs" "${INTERSHEET_REFS}"
+			(at 213.36 95.4892 90)
+			(effects
+				(font
+					(size 1.27 1.27)
+				)
+				(justify left)
+				(hide yes)
+			)
+		)
+	)
 	(global_label "VBUS"
 		(shape input)
@@
 	(global_label "ADC"
 		(shape output)
-		(at 90.17 130.175 0)
+		(at 89.535 142.24 0)
 		(effects
 			(font
@@
 		)
 		(property "Intersheetrefs" "${INTERSHEET_REFS}"
-			(at 90.17 130.175 0)
+			(at 89.535 142.24 0)
 			(effects
 				(font
@@
 		)
 	)
-	(global_label "VBAT"
+	(global_label "VSWITCHED"
 		(shape output)
 		(at 263.525 118.745 0)
@@
 		)
 		(property "Intersheetrefs" "${INTERSHEET_REFS}"
-			(at 270.2708 118.745 0)
+			(at 276.1974 118.745 0)
 			(effects
 				(font
@@
 		)
 	)
-	(global_label "VBAT"
+	(global_label "VSWITCHED"
 		(shape input)
 		(at 158.75 29.845 180)
@@
 		)
 		(property "Intersheetrefs" "${INTERSHEET_REFS}"
-			(at 152.0042 29.845 0)
+			(at 146.0776 29.845 0)
 			(effects
 				(font
@@
 		)
 	)
-	(global_label "VBAT"
+	(global_label "VSWITCHED"
 		(shape input)
-		(at 86.36 114.935 90)
+		(at 85.725 127 90)
 		(fields_autoplaced yes)
 		(effects
@@
 		)
 		(property "Intersheetrefs" "${INTERSHEET_REFS}"
-			(at 86.36 108.1892 90)
+			(at 85.725 114.3276 90)
 			(effects
 				(font
@@
 	(global_label "ADCL"
 		(shape bidirectional)
-		(at 86.36 137.795 270)
+		(at 85.725 149.86 270)
 		(effects
 			(font
@@
 		)
 		(property "Intersheetrefs" "${INTERSHEET_REFS}"
-			(at 86.36 137.795 90)
+			(at 85.725 149.86 90)
 			(effects
 				(font
@@
 	(symbol
 		(lib_id "Device:R")
-		(at 86.36 133.985 0)
+		(at 85.725 146.05 0)
 		(unit 1)
 		(exclude_from_sim no)
@@
 		(dnp no)
 		(property "Reference" "R7"
-			(at 86.36 133.985 90)
+			(at 85.725 146.05 90)
 			(effects
 				(font
@@
 		)
 		(property "Value" "100K 1%"
-			(at 88.9 135.89 90)
+			(at 88.265 147.955 90)
 			(effects
 				(font
@@
 		)
 		(property "Footprint" "RevK:R_0402"
-			(at 84.582 133.985 90)
+			(at 83.947 146.05 90)
 			(effects
 				(font
@@
 		)
 		(property "Datasheet" "~"
-			(at 86.36 133.985 0)
+			(at 85.725 146.05 0)
 			(effects
 				(font
@@
 		)
 		(property "Description" "Resistor"
-			(at 86.36 133.985 0)
+			(at 85.725 146.05 0)
 			(effects
 				(font
@@
 		)
 		(property "MPN" "C5139597"
-			(at 86.36 133.985 90)
+			(at 85.725 146.05 90)
 			(effects
 				(font
@@
 	)
 	(symbol
-		(lib_id "power:PWR_FLAG")
-		(at 213.36 105.41 0)
-		(unit 1)
-		(exclude_from_sim no)
-		(in_bom yes)
-		(on_board yes)
-		(dnp no)
-		(fields_autoplaced yes)
-		(property "Reference" "#FLG04"
-			(at 213.36 103.505 0)
-			(effects
-				(font
-					(size 1.27 1.27)
-				)
-				(hide yes)
-			)
-		)
-		(property "Value" "PWR_FLAG"
-			(at 213.36 101.2769 0)
-			(effects
-				(font
-					(size 1.27 1.27)
-				)
-			)
-		)
-		(property "Footprint" ""
-			(at 213.36 105.41 0)
-			(effects
-				(font
-					(size 1.27 1.27)
-				)
-				(hide yes)
-			)
-		)
-		(property "Datasheet" "~"
-			(at 213.36 105.41 0)
-			(effects
-				(font
-					(size 1.27 1.27)
-				)
-				(hide yes)
-			)
-		)
-		(property "Description" "Special symbol for telling ERC where power comes from"
-			(at 213.36 105.41 0)
-			(effects
-				(font
-					(size 1.27 1.27)
-				)
-				(hide yes)
-			)
-		)
-		(pin "1"
-		)
-		(instances
-			(project "Gyro"
-				(path "/babeabf2-f3b0-4ed5-8d9e-0215947e6cf3"
-					(reference "#FLG04")
-					(unit 1)
-				)
-			)
-		)
-	)
-	(symbol
 		(lib_id "Device:C")
 		(at 59.055 142.24 0)
@@
 	(symbol
 		(lib_id "Device:R")
-		(at 86.36 126.365 0)
+		(at 85.725 138.43 0)
 		(unit 1)
 		(exclude_from_sim no)
@@
 		(dnp no)
 		(property "Reference" "R6"
-			(at 86.36 126.365 90)
+			(at 85.725 138.43 90)
 			(effects
 				(font
@@
 		)
 		(property "Value" "100K 1%"
-			(at 83.82 125.73 90)
+			(at 83.185 137.795 90)
 			(effects
 				(font
@@
 		)
 		(property "Footprint" "RevK:R_0402"
-			(at 84.582 126.365 90)
+			(at 83.947 138.43 90)
 			(effects
 				(font
@@
 		)
 		(property "Datasheet" "~"
-			(at 86.36 126.365 0)
+			(at 85.725 138.43 0)
 			(effects
 				(font
@@
 		)
 		(property "Description" "Resistor"
-			(at 86.36 126.365 0)
+			(at 85.725 138.43 0)
 			(effects
 				(font
@@
 		)
 		(property "MPN" "C5139597"
-			(at 86.36 126.365 90)
+			(at 85.725 138.43 90)
 			(effects
 				(font
@@
 	(symbol
 		(lib_id "Device:R")
-		(at 86.36 118.745 0)
+		(at 85.725 130.81 0)
 		(unit 1)
 		(exclude_from_sim no)
@@
 		(dnp no)
 		(property "Reference" "R5"
-			(at 86.36 118.745 90)
+			(at 85.725 130.81 90)
 			(effects
 				(font
@@
 		)
 		(property "Value" "100K 1%"
-			(at 88.9 118.11 90)
+			(at 88.265 130.175 90)
 			(effects
 				(font
@@
 		)
 		(property "Footprint" "RevK:R_0402"
-			(at 84.582 118.745 90)
+			(at 83.947 130.81 90)
 			(effects
 				(font
@@
 		)
 		(property "Datasheet" "~"
-			(at 86.36 118.745 0)
+			(at 85.725 130.81 0)
 			(effects
 				(font
@@
 		)
 		(property "Description" "Resistor"
-			(at 86.36 118.745 0)
+			(at 85.725 130.81 0)
 			(effects
 				(font
@@
 		)
 		(property "MPN" "C5139597"
-			(at 86.36 118.745 90)
+			(at 85.725 130.81 90)
 			(effects
 				(font
